File: mykeyboard/mykeyboard.kicad_pcb (KiCad board)
At the start: 2 copper layers, 285.7 x 113.5 mm, 176 parts, among them J3 Debug, K0 ~~,`, K1 !,1, K10 ),0, K11 _,-, K12 +,=, K13 Backspace, K14 Tab, K15 Q, K16 W, K17 E, K18 R, K19 T, K2 @,2, K20 Y, K21 U, K22 I, K23 O, K24 P, K25 {,[, K26 },], K27 |,\, K28 Caps Lock, K29 A, K3 #,3, K30 S, K31 D, K32 F, K33 G, K34 H, K35 J, K36 K, K37 L, K38 :,;, K39 ",', K4 $,4, K40 Enter, K41 Shift, K42 Z, K43 X, K44 C, K45 V, K46 B, K47 N, K48 M, K49 <,,, K5 %,5, K50 >,., K51 ?,/, K52 Shift, K53 Ctrl, K54 Win, K55 Alt, K56 Blank, K57 Alt, K58 Win, K59 Menu, K6 ^,6, K60 Ctrl, K7 &,7, K8 *,8, K9 (,9, P1 USB-C, SW1 Reset, U1 BQ21040DBVR, U2 nRF52840, U3 ESDR0502NMUTAG, Y1 32.768 kHz, Y2 32MHz

Commit message: ITSY CHANGE
Other:
- board outline removed
Changed lines of the file:
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@@
 			(type solid)
 		)
-		(layer "Edge.Cuts")
+		(layer "Margin")
 	)
 	(gr_arc
@@
 			(type solid)
 		)
-		(layer "Edge.Cuts")
+		(layer "Margin")
 	)
 	(gr_line
@@
 			(type solid)
 		)
-		(layer "Edge.Cuts")
+		(layer "Margin")
 	)
 	(gr_line
@@
 			(type solid)
 		)
-		(layer "Edge.Cuts")
+		(layer "Margin")
 	)
 	(gr_arc
@@
 			(type solid)
 		)
-		(layer "Edge.Cuts")
+		(layer "Margin")
 	)
 	(gr_line
@@
 			(type solid)
 		)
-		(layer "Edge.Cuts")
+		(layer "Margin")
 	)
 	(gr_arc
@@
 			(type solid)
 		)
-		(layer "Edge.Cuts")
+		(layer "Margin")
 	)
 	(gr_arc
@@
 			(type solid)
 		)
-		(layer "Edge.Cuts")
+		(layer "Margin")
 	)
 	(gr_text "HACKCLUB"
